Commit message: fix: HE-2495-change-gripper-side

File: code/softenable.urdf (robot description, URDF)
Before this commit: robot softenable, 41 links, 40 joints
Links:
- removed link placement_link
- added link left_placement_link
- added link right_placement_link
Joints:
- added joint right_tip_placement: type fixed, parent dlr_gripper_center, child right_placement_link, origin xyz=0.0 -0.025 0.1 rpy=0.0 0.0 3.141592653589793
- joint left_tip_placement: child placement_link -> left_placement_link
